File: electronics/rev2/ecad/Multimeter.kicad_pcb (KiCad board)
At the start: 2 copper layers, 68 x 110 mm, 68 parts, among them J3 Red Banana Plug, J4 Black Banana Plug, Q1 2N7002, Q12 2N7002, Q14 2N7002, Q15 2N7002, Q16 2N7002, Q2 2N7002, Q3 2N7002, Q4 2N7002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

Commit message: display doing stuff
Parts:
- added R21: 100k+/-0.1%, Resistor_SMD:R_0805_2012Metric_Pad1.20x1.40mm_HandSolder, F.Cu at (116.6, 120.9)
- added R22: 10k, Resistor_SMD:R_0805_2012Metric_Pad1.20x1.40mm_HandSolder, F.Cu at (116.6, 124.4)
- added SW2: GF-126-0159, Multimeter:SW_GF-126-0159, F.Cu at (127.4, 121.0)
- added TP4: 4952, Connector_Pin:Pin_D1.2mm_L10.2mm_W2.9mm_FlatFork, F.Cu at (171.8, 115.4)
- R38: value 1.5M+/-0.1% -> 10k+/-0.1%
- TP1, TP2, TP3: value 4952 -> Pad
- moved R3 12.3 mm to (139.0, 133.0)
- moved SW1 12.0 mm to (127.4, 133.1)
- moved TP3 6.77 mm to (130.1, 79.3)
- moved R38 1.08 mm to (117.4, 113.0), turned to 90 degrees
- renumbered S1 to SW3
Connections:
- R38 pad 1: Net-(U3A--) -> Net-(SW2A-A)
- TP3 pad 1: Net-(U3A--) -> Net-(SW2A-B)
- U1 pad 11: unconnected-(U1-GP8-Pad11) -> /Analog Front End/RANGE
- U3 pad 1: Net-(U3A--) -> Net-(SW2A-B)
- U3 pad 2: Net-(U3A--) -> Net-(SW2A-B)
Routing:
- net Net-(U3A--): track 70.7 -> 0.00 mm
- net Net-(SW2A-B): track 0.00 -> 63.7 mm, vias 0 -> 6
- net /Analog Front End/RANGE: track 0.00 -> 44.9 mm, vias 0 -> 4
- net Net-(SW2A-C): track 0.00 -> 16.9 mm
- net Net-(R21-Pad2): track 4.81 -> 15.7 mm
- net Net-(SW2A-A): track 0.00 -> 7.82 mm
- net Net-(SW2B-A): track 0.00 -> 5.24 mm
- net Net-(SW1-B): track 54.5 -> 50.8 mm
- net GND: track 83.1 -> 84.4 mm
- net +3.3V: track 56.6 -> 55.4 mm, vias 12 -> 10
Other:
- board text added: "low Ω/Neg"
- board text added: "trig"
- board text removed: "low Ω"
- board text removed: "pico"

Commit message: ordered some stuff
Parts:
- removed C1: 0.1uF, Capacitor_SMD:C_0805_2012Metric
- removed R7, R8: 10k, Resistor_SMD:R_0805_2012Metric_Pad1.20x1.40mm_HandSolder
- removed U5: MCP23008-xSO, Package_SO:SOIC-18W_7.5x11.6mm_P1.27mm
- added Q10: BSS84, Package_TO_SOT_SMD:SOT-23, F.Cu at (148.6, 61.4)
- added Q11: BSS84, Package_TO_SOT_SMD:SOT-23, F.Cu at (152.2, 61.4)
- added Q13: BSS84, Package_TO_SOT_SMD:SOT-23, F.Cu at (141.5, 61.4)
- added Q17: 2N7002, Package_TO_SOT_SMD:SOT-23, F.Cu at (157.8, 66.6)
- added Q18: 2N7002, Package_TO_SOT_SMD:SOT-23, F.Cu at (154.2, 66.7)
- added Q19: 2N7002, Package_TO_SOT_SMD:SOT-23, F.Cu at (143.6, 66.7)
- added Q20: 2N7002, Package_TO_SOT_SMD:SOT-23, F.Cu at (136.5, 66.7)
- added Q21: 2N7002, Package_TO_SOT_SMD:SOT-23, F.Cu at (132.9, 66.7)
- added Q22: 2N7002, Package_TO_SOT_SMD:SOT-23, F.Cu at (147.2, 66.7)
- added Q23: 2N7002, Package_TO_SOT_SMD:SOT-23, F.Cu at (150.7, 66.7)
- added Q24: 2N7002, Package_TO_SOT_SMD:SOT-23, F.Cu at (140.0, 66.7)
- added Q5: BSS84, Package_TO_SOT_SMD:SOT-23, F.Cu at (159.4, 61.3)
- added Q6: BSS84, Package_TO_SOT_SMD:SOT-23, F.Cu at (155.8, 61.4)
- added Q7: BSS84, Package_TO_SOT_SMD:SOT-23, F.Cu at (145.0, 61.4)
- added Q8: BSS84, Package_TO_SOT_SMD:SOT-23, F.Cu at (137.9, 61.4)
- added Q9: BSS84, Package_TO_SOT_SMD:SOT-23, F.Cu at (134.2, 61.4)
- added R23: 10k, Resistor_SMD:R_0805_2012Metric_Pad1.20x1.40mm_HandSolder, F.Cu at (155.8, 71.9)
- added R24: 10k, Resistor_SMD:R_0805_2012Metric_Pad1.20x1.40mm_HandSolder, F.Cu at (143.7, 71.9)
- added R25: 10k, Resistor_SMD:R_0805_2012Metric_Pad1.20x1.40mm_HandSolder, F.Cu at (135.6, 71.9)
- added R26: 10k, Resistor_SMD:R_0805_2012Metric_Pad1.20x1.40mm_HandSolder, F.Cu at (131.6, 71.9)
- added R27: 10k, Resistor_SMD:R_0805_2012Metric_Pad1.20x1.40mm_HandSolder, F.Cu at (147.7, 71.9)
- added R43: 10k, Resistor_SMD:R_0805_2012Metric_Pad1.20x1.40mm_HandSolder, F.Cu at (151.8, 71.9)
- added R44: 10k, Resistor_SMD:R_0805_2012Metric_Pad1.20x1.40mm_HandSolder, F.Cu at (139.6, 71.9)
- added R45: 1k, Resistor_SMD:R_0805_2012Metric_Pad1.20x1.40mm_HandSolder, F.Cu at (157.8, 71.9)
- added R46: 1k, Resistor_SMD:R_0805_2012Metric_Pad1.20x1.40mm_HandSolder, F.Cu at (153.8, 71.9)
- added R47: 1k, Resistor_SMD:R_0805_2012Metric_Pad1.20x1.40mm_HandSolder, F.Cu at (141.7, 71.9)
- added R48: 1k, Resistor_SMD:R_0805_2012Metric_Pad1.20x1.40mm_HandSolder, F.Cu at (133.6, 71.9)
- added R49: 1k, Resistor_SMD:R_0805_2012Metric_Pad1.20x1.40mm_HandSolder, F.Cu at (129.6, 71.9)
- added R50: 1k, Resistor_SMD:R_0805_2012Metric_Pad1.20x1.40mm_HandSolder, F.Cu at (145.7, 71.9)
- added R51: 1k, Resistor_SMD:R_0805_2012Metric_Pad1.20x1.40mm_HandSolder, F.Cu at (149.7, 71.9)
- added R52: 1k, Resistor_SMD:R_0805_2012Metric_Pad1.20x1.40mm_HandSolder, F.Cu at (137.6, 71.9)
- moved R6 5.48 mm to (159.9, 71.9), turned to 90 degrees
- moved TP1 3.20 mm to (154.2, 81.3)
- moved U3 2.40 mm to (149.1, 84.4)
- moved C4 2.04 mm to (143.6, 84.0)
- moved R36 1.73 mm to (142.1, 87.2)
- moved U7 1.73 mm to (139.3, 87.4)
- moved TP3 1.10 mm to (130.1, 80.4)
Connections:
- U1 pad 24: unconnected-(U1-GP18-Pad24) -> /Display/DP
- U1 pad 25: unconnected-(U1-GP19-Pad25) -> /Display/G
- U1 pad 26: unconnected-(U1-GP20-Pad26) -> /Display/F
- U1 pad 27: unconnected-(U1-GP21-Pad27) -> /Display/E
- U1 pad 29: unconnected-(U1-GP22-Pad29) -> /Display/D
- U1 pad 31: /Display/SDA -> /Display/C
- U1 pad 32: /Display/SCL -> /Display/B
- U1 pad 34: unconnected-(U1-GP28-Pad34) -> /Display/A
Routing:
- net /Display/SDA: track 101.0 -> 0.00 mm, vias 4 -> 0
- net /Display/SCL: track 91.4 -> 0.00 mm, vias 6 -> 0
- net /Display/D: track 0.00 -> 82.4 mm, vias 0 -> 2
- net /Display/C: track 0.00 -> 82.3 mm, vias 0 -> 2
- net /Display/E: track 0.00 -> 79.8 mm, vias 0 -> 2
- net /Display/A: track 0.00 -> 79.6 mm, vias 0 -> 2
- net /Display/B: track 0.00 -> 78.1 mm, vias 0 -> 2
- net /Display/DP: track 0.00 -> 70.5 mm, vias 0 -> 2
- net /Display/F: track 0.00 -> 69.1 mm, vias 0 -> 2
- net /Display/G: track 0.00 -> 65.2 mm, vias 0 -> 2
- net +5V: track 126.7 -> 149.9 mm, vias 8 -> 14
- net Net-(Q9-D): track 17.3 -> 2.29 mm
- net Net-(Q8-D): track 14.9 -> 2.16 mm
- net GND: track 84.4 -> 96.5 mm, vias 33 -> 38
- net Net-(Q18-D): track 0.00 -> 9.95 mm
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
Commit message: rev2 cal
Parts:
- R38, R5: value 10k+/-0.1% -> 649
