File: electronics/rev2/ecad/Multimeter.kicad_sch (KiCad schematic)
At the start: 9 parts, among them SW1 GF-123-0054, U1 SC0915

Commit message: export
Parts:
- R3: Digikey Part # RMCF0805FT10K0CT-ND -> 311-10.0KCRCT-ND; Part # RMCF0805FT10K0 -> RC0805FR-0710KL
- R7, R8: Digikey Part # (none) -> 311-10.0KCRCT-ND; Part # (none) -> RC0805FR-0710KL; Unit Price (none) -> 0.1
Changed lines of the file:
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@@
 	(title_block
 		(title "Multimeter")
+		(date "2024-03-03")
 		(rev "1")
 	)
@@
 			)
 		)
+		(property "Digikey Part #" "311-10.0KCRCT-ND"
+			(at 166.37 88.9 0)
+			(effects
+				(font
+					(size 1.27 1.27)
+				)
+				(hide yes)
+			)
+		)
+		(property "Part #" "RC0805FR-0710KL"
+			(at 166.37 88.9 0)
+			(effects
+				(font
+					(size 1.27 1.27)
+				)
+				(hide yes)
+			)
+		)
+		(property "Unit Price" "0.1"
+			(at 166.37 88.9 0)
+			(effects
+				(font
+					(size 1.27 1.27)
+				)
+				(hide yes)
+			)
+		)
 		(pin "2"
 		)
@@
 			)
 		)
+		(property "Digikey Part #" "311-10.0KCRCT-ND"
+			(at 176.53 88.9 0)
+			(effects
+				(font
+					(size 1.27 1.27)
+				)
+				(hide yes)
+			)
+		)
+		(property "Part #" "RC0805FR-0710KL"
+			(at 176.53 88.9 0)
+			(effects
+				(font
+					(size 1.27 1.27)
+				)
+				(hide yes)
+			)
+		)
+		(property "Unit Price" "0.1"
+			(at 176.53 88.9 0)
+			(effects
+				(font
+					(size 1.27 1.27)
+				)
+				(hide yes)
+			)
+		)
 		(pin "2"
 		)
@@
 			)
 		)
-		(property "Digikey Part #" "RMCF0805FT10K0CT-ND"
+		(property "Digikey Part #" "311-10.0KCRCT-ND"
 			(at 77.47 40.64 0)
 			(effects
@@
 			)
 		)
-		(property "Part #" "RMCF0805FT10K0"
+		(property "Part #" "RC0805FR-0710KL"
 			(at 77.47 40.64 0)
 			(effects

Commit message: display doing stuff
Parts:
- added TP4: 4952, Connector_Pin:Pin_D1.2mm_L10.2mm_W2.9mm_FlatFork, symbol Connector:TestPoint
- R3, R7, R8: Digikey Part # 311-10.0KCRCT-ND -> RMCF0805FT10K0CT-ND; Part # RC0805FR-0710KL -> RMCF0805FT10K0
Connections:
- net GND: now also TP4.1
- net Analog Front End/RANGE: now reaches U1.11 (GP8)
- no-connect marks 20 -> 19
Other:
- sheet Analog Front End ports: added RANGE; removed none
- note added: "GND Test Point"
Changed lines of the file:
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@@
+	)
+	(junction
+		(at 125.73 138.43)
+		(diameter 0)
+		(color 0 0 0 0)
 	)
 	(junction
@@
 	)
 	(no_connect
-		(at 109.22 88.9)
-	)
-	(no_connect
 		(at 160.02 86.36)
 	)
@@
 	(wire
 		(pts
-			(xy 168.91 149.86) (xy 100.33 149.86)
+			(xy 168.91 158.75) (xy 100.33 158.75)
 		)
 		(stroke
@@
 	(wire
 		(pts
-			(xy 167.64 104.14) (xy 167.64 148.59)
+			(xy 167.64 104.14) (xy 167.64 157.48)
 		)
 		(stroke
@@
 	(wire
 		(pts
+			(xy 125.73 138.43) (xy 125.73 146.05)
+		)
+		(stroke
+			(width 0)
+			(type default)
+		)
+	)
+	(wire
+		(pts
 			(xy 107.95 114.3) (xy 109.22 114.3)
 		)
@@
 	(wire
 		(pts
-			(xy 171.45 111.76) (xy 171.45 152.4)
+			(xy 171.45 111.76) (xy 171.45 161.29)
 		)
 		(stroke
@@
 	(wire
 		(pts
-			(xy 100.33 149.86) (xy 100.33 96.52)
+			(xy 100.33 158.75) (xy 100.33 96.52)
 		)
 		(stroke
@@
 	(wire
 		(pts
-			(xy 170.18 109.22) (xy 170.18 151.13)
+			(xy 170.18 109.22) (xy 170.18 160.02)
 		)
 		(stroke
@@
 	(wire
 		(pts
-			(xy 171.45 152.4) (xy 97.79 152.4)
+			(xy 171.45 161.29) (xy 97.79 161.29)
 		)
 		(stroke
@@
 	(wire
 		(pts
-			(xy 101.6 148.59) (xy 101.6 99.06)
+			(xy 101.6 157.48) (xy 101.6 99.06)
 		)
 		(stroke
@@
 	(wire
 		(pts
-			(xy 167.64 148.59) (xy 101.6 148.59)
-		)
-		(stroke
-			(width 0)
-			(type default)
-		)
-	)
-	(wire
-		(pts
-			(xy 99.06 151.13) (xy 99.06 93.98)
+			(xy 167.64 157.48) (xy 101.6 157.48)
+		)
+		(stroke
+			(width 0)
+			(type default)
+		)
+	)
+	(wire
+		(pts
+			(xy 99.06 160.02) (xy 99.06 93.98)
 		)
 		(stroke
@@
 	(wire
 		(pts
-			(xy 97.79 152.4) (xy 97.79 91.44)
+			(xy 97.79 161.29) (xy 97.79 91.44)
 		)
 		(stroke
@@
 	(wire
 		(pts
-			(xy 170.18 151.13) (xy 99.06 151.13)
+			(xy 95.25 88.9) (xy 109.22 88.9)
+		)
+		(stroke
+			(width 0)
+			(type default)
+		)
+	)
+	(wire
+		(pts
+			(xy 170.18 160.02) (xy 99.06 160.02)
 		)
 		(stroke
@@
 	(wire
 		(pts
-			(xy 168.91 106.68) (xy 168.91 149.86)
+			(xy 168.91 106.68) (xy 168.91 158.75)
 		)
 		(stroke
@@
 			)
 			(justify left top)
+		)
+	)
+	(text "GND Test Point"
+		(exclude_from_sim no)
+		(at 126.492 153.416 0)
+		(effects
+			(font
+				(size 1.27 1.27)
+			)
 		)
 	)
@@
 	)
 	(symbol
+		(lib_id "Connector:TestPoint")
+		(at 125.73 146.05 180)
+		(unit 1)
+		(exclude_from_sim no)
+		(in_bom yes)
+		(on_board yes)
+		(dnp no)
+		(fields_autoplaced yes)
+		(property "Reference" "TP4"
+			(at 128.27 148.0819 0)
+			(effects
+				(font
+					(size 1.27 1.27)
+				)
+				(justify right)
+			)
+		)
+		(property "Value" "4952"
+			(at 128.27 150.6219 0)
+			(effects
+				(font
+					(size 1.27 1.27)
+				)
+				(justify right)
+			)
+		)
+		(property "Footprint" "Connector_Pin:Pin_D1.2mm_L10.2mm_W2.9mm_FlatFork"
+			(at 120.65 146.05 0)
+			(effects
+				(font
+					(size 1.27 1.27)
+				)
+				(hide yes)
+			)
+		)
+		(property "Datasheet" "~"
+			(at 120.65 146.05 0)
+			(effects
+				(font
+					(size 1.27 1.27)
+				)
+				(hide yes)
+			)
+		)
+		(property "Description" "test point"
+			(at 125.73 146.05 0)
+			(effects
+				(font
+					(size 1.27 1.27)
+				)
+				(hide yes)
+			)
+		)
+		(property "Digikey Part #" "36-4952-ND"
+			(at 125.73 146.05 0)
+			(effects
+				(font
+					(size 1.27 1.27)
+				)
+				(hide yes)
+			)
+		)
+		(property "Part #" "4952"
+			(at 125.73 146.05 0)
+			(effects
+				(font
+					(size 1.27 1.27)
+				)
+				(hide yes)
+			)
+		)
+		(property "Unit Price" "0.26"
+			(at 125.73 146.05 0)
+			(effects
+				(font
+					(size 1.27 1.27)
+				)
+				(hide yes)
+			)
+		)
+		(pin "1"
+		)
+		(instances
+			(project "Multimeter"
+				(path "/cb819000-1954-426e-958e-510a70bc03c7"
+					(reference "TP4")
+					(unit 1)
+				)
+			)
+		)
+	)
+	(symbol
 		(lib_id "power:GND")
 		(at 107.95 115.57 0)
@@
 			)
 		)
-		(property "Digikey Part #" "311-10.0KCRCT-ND"
+		(property "Digikey Part #" "RMCF0805FT10K0CT-ND"
 			(at 166.37 88.9 0)
 			(effects
@@
 			)
 		)
-		(property "Part #" "RC0805FR-0710KL"
+		(property "Part #" "RMCF0805FT10K0"
 			(at 166.37 88.9 0)
 			(effects
@@
 			)
 		)
-		(property "Digikey Part #" "311-10.0KCRCT-ND"
+		(property "Digikey Part #" "RMCF0805FT10K0CT-ND"
 			(at 176.53 88.9 0)
 			(effects
@@
 			)
 		)
-		(property "Part #" "RC0805FR-0710KL"
+		(property "Part #" "RMCF0805FT10K0"
 			(at 176.53 88.9 0)
 			(effects
@@
 			)
 		)
-		(property "Digikey Part #" "311-10.0KCRCT-ND"
+		(property "Digikey Part #" "RMCF0805FT10K0CT-ND"
 			(at 77.47 40.64 0)
 			(effects
@@
 			)
 		)
-		(property "Part #" "RC0805FR-0710KL"
+		(property "Part #" "RMCF0805FT10K0"
 			(at 77.47 40.64 0)
 			(effects
@@
 			(effects
 				(font
+					(size 1.27 1.27)
+				)
+				(justify right)
+			)
+		)
+		(pin "RANGE" output
+			(at 95.25 88.9 0)
+			(effects
+				(font

Commit message: ordered some stuff
Parts:
- removed R7, R8: 10k, Resistor_SMD:R_0805_2012Metric_Pad1.20x1.40mm_HandSolder, symbol Device:R_US
Connections:
- net Display/DP: now reaches U1.24 (GP18)
- net Display/G: now reaches U1.25 (GP19)
- net Display/F: now reaches U1.26 (GP20)
- net Display/E: now reaches U1.27 (GP21)
- net Display/D: now reaches U1.29 (GP22)
- net Display/A: now reaches U1.34 (GP28)
- net Display/SCL renamed Display/B
- net Display/SDA renamed Display/C
- no-connect marks 19 -> 13
Other:
- sheet Display ports: added A, B, C, D, DP, E, F, G; removed SCL, SDA

Commit message: rev2 cal
Parts:
- U1: Availability (none) -> In Stock; Check_prices (none) -> https://www.snapeda.com/parts/SC0915/Raspberry+Pi/view-part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; MANUFACTURER (none) -> Pi Supply; MF (none) -> Raspberry Pi; MP (none) -> SC0915; PARTREV (none) -> 1.9; Package (none) -> None; Price (none) -> None; Purchase-URL (none) -> https://www.snapeda.com/api/url_track_click_mouser/?unipart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; SNAPEDA_PN (none) -> SC0915; STANDARD (none) -> Manufacturer Recommendations; SnapEDA_Link (none) -> https://www.snapeda.com/parts/SC0915/Raspberry+Pi/view-part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
Changed lines of the file:
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@@
 			)
 		)
-		(property "Description" ""
+		(property "Description" "Mounting Hole with connection"
 			(at 250.19 140.97 0)
 			(effects
@@
 			)
 		)
-		(property "Description" ""
+		(property "Description" "Power symbol creates a global label with name \"+3.3V\""
 			(at 173.99 49.53 0)
 			(effects
@@
 			)
 		)
-		(property "Description" ""
+		(property "Description" "Power symbol creates a global label with name \"+3.3V\""
 			(at 68.58 35.56 0)
 			(effects
@@
 			)
 		)
-		(property "Description" ""
+		(property "Description" "Power symbol creates a global label with name \"GND\" , ground"
 			(at 250.19 144.78 0)
 			(effects
@@
 			)
 		)
-		(property "Description" ""
+		(property "Description" "Power symbol creates a global label with name \"GND\" , ground"
 			(at 134.62 139.7 0)
 			(effects
@@
 			)
 		)
-		(property "Description" ""
+		(property "Description" "\nRaspberry Pi Pico Embedded Dev Module | Raspberry Pi SC0915\n"
 			(at 134.62 88.9 0)
 			(effects
@@
 			)
 		)
-		(property "Price" ""
+		(property "Price" "None"
 			(at 134.62 88.9 0)
 			(effects
@@
 			)
 		)
+		(property "MF" "Raspberry Pi"
+			(at 134.62 88.9 0)
+			(effects
+				(font
+					(size 1.27 1.27)
+				)
+				(justify bottom)
+				(hide yes)
+			)
+		)
+		(property "Package" "None"
+			(at 134.62 88.9 0)
+			(effects
+				(font
+					(size 1.27 1.27)
+				)
+				(justify bottom)
+				(hide yes)
+			)
+		)
+		(property "Check_prices" "https://www.snapeda.com/parts/SC0915/Raspberry+Pi/view-part/?ref=eda"
+			(at 134.62 88.9 0)
+			(effects
+				(font
+					(size 1.27 1.27)
+				)
+				(justify bottom)
+				(hide yes)
+			)
+		)
+		(property "STANDARD" "Manufacturer Recommendations"
+			(at 134.62 88.9 0)
+			(effects
+				(font
+					(size 1.27 1.27)
+				)
+				(justify bottom)
+				(hide yes)
+			)
+		)
+		(property "PARTREV" "1.9"
+			(at 134.62 88.9 0)
+			(effects
+				(font
+					(size 1.27 1.27)
+				)
+				(justify bottom)
+				(hide yes)
+			)
+		)
+		(property "SnapEDA_Link" "https://www.snapeda.com/parts/SC0915/Raspberry+Pi/view-part/?ref=snap"
+			(at 134.62 88.9 0)
+			(effects
+				(font
+					(size 1.27 1.27)
+				)
+				(justify bottom)
+				(hide yes)
+			)
+		)
+		(property "MP" "SC0915"
+			(at 134.62 88.9 0)
+			(effects
+				(font
+					(size 1.27 1.27)
+				)
+				(justify bottom)
+				(hide yes)
+			)
+		)
+		(property "Purchase-URL" "https://www.snapeda.com/api/url_track_click_mouser/?unipart_id=6331605&manufacturer=Raspberry Pi&part_name=SC0915&search_term=raspberry pi pico"
+			(at 134.62 88.9 0)
+			(effects
+				(font
+					(size 1.27 1.27)
+				)
+				(justify bottom)
+				(hide yes)
+			)
+		)
+		(property "MANUFACTURER" "Pi Supply"
+			(at 134.62 88.9 0)
+			(effects
+				(font
+					(size 1.27 1.27)
+				)
+				(justify bottom)
+				(hide yes)
+			)
+		)
+		(property "Availability" "In Stock"
+			(at 134.62 88.9 0)
+			(effects
+				(font
+					(size 1.27 1.27)
+				)
+				(justify bottom)
+				(hide yes)
+			)
+		)
+		(property "SNAPEDA_PN" "SC0915"
+			(at 134.62 88.9 0)
+			(effects
+				(font
+					(size 1.27 1.27)
+				)
+				(justify bottom)
+				(hide yes)
+			)
+		)
 		(pin "40"
 		)
@@
 			)
 		)
-		(property "Description" ""
+		(property "Description" "Power symbol creates a global label with name \"GND\" , ground"
 			(at 107.95 115.57 0)
 			(effects
@@
 			)
 		)
-		(property "Description" ""
+		(property "Description" "Power symbol creates a global label with name \"GND\" , ground"
 			(at 250.19 160.02 0)
 			(effects
@@
 			)
 		)
-		(property "Description" ""
+		(property "Description" "Mounting Hole with connection"
 			(at 250.19 156.21 0)
 			(effects
@@
 			)
 		)
-		(property "Description" ""
+		(property "Description" "Power symbol creates a global label with name \"GND\" , ground"
 			(at 161.29 128.27 0)
 			(effects
@@
 			)
 		)
-		(property "Description" ""
+		(property "Description" "Power symbol creates a global label with name \"GND\" , ground"
 			(at 82.55 53.34 0)
 			(effects
@@
 			)
 		)
-		(property "Description" ""
+		(property "Description" "Mounting Hole with connection"
 			(at 238.76 140.97 0)
 			(effects
@@
 			)
 		)
-		(property "Description" ""
+		(property "Description" "Power symbol creates a global label with name \"GND\" , ground"
 			(at 238.76 144.78 0)
 			(effects
@@
 			)
 		)
-		(property "Description" ""
+		(property "Description" "Power symbol creates a global label with name \"GND\" , ground"
 			(at 238.76 160.02 0)
 			(effects
@@
 			)
 		)
-		(property "Description" ""
+		(property "Description" "Mounting Hole with connection"
 			(at 238.76 156.21 0)
 			(effects
@@
 			)
 		)
-		(property "Description" ""
+		(property "Description" "Special symbol for telling ERC where power comes from"
 			(at 184.15 49.53 0)
 			(effects
@@
 			)
 		)
-		(property "Description" ""
+		(property "Description" "Special symbol for telling ERC where power comes from"
 			(at 163.83 39.37 0)
 			(effects
@@
 			)
 		)
-		(property "Description" ""
+		(property "Description" "Single Pole Single Throw (SPST) switch"
 			(at 82.55 46.99 0)
 			(effects
@@
 			)
 		)
-		(property "Description" ""
+		(property "Description" "Power symbol creates a global label with name \"+5V\""
 			(at 168.91 44.45 0)
 			(effects
@@
 			)
 		)
-		(property "Description" ""
+		(property "Description" "Resistor, US symbol"
 			(at 77.47 40.64 0)
 			(effects
