File: electronics/rev3/ecad/Multimeter.kicad_pcb (KiCad board)
At the start: 2 copper layers, 68 x 110 mm, 99 parts, among them J3 Red Banana Plug, J4 Black Banana Plug, Q1 2N7002, Q10 BSS84, Q11 BSS84, Q12 2N7002, Q13 BSS84, Q14 2N7002, Q15 2N7002, Q16 2N7002, Q17 2N7002, Q18 2N7002, Q19 2N7002, Q2 2N7002, Q20 2N7002, Q21 2N7002, Q22 2N7002, Q23 2N7002, Q24 2N7002, Q3 2N7002, Q4 2N7002, Q5 BSS84, Q6 BSS84, Q7 BSS84, Q8 BSS84, Q9 BSS84, SW1 GF-123-0054, SW2 GF-126-0159, SW3 GF-161-0005, U1 SC0915, U10 MCP3561, U3 OPA4388IDR, U4 CC56-12SURKWA, U7 LM4030-2.5

Commit message: layout work rev3
Parts:
- removed SW2: GF-126-0159, Multimeter:SW_GF-126-0159
- removed U7: LM4030-2.5, Package_TO_SOT_SMD:SOT-23-5
- added C1: 1uF, Capacitor_SMD:C_0805_2012Metric, F.Cu at (133.4, 115.2)
- added C13: 0.1uF, Capacitor_SMD:C_0805_2012Metric, F.Cu at (140.9, 117.0)
- added C14: 10nF, Capacitor_SMD:C_0805_2012Metric, F.Cu at (148.1, 116.2)
- added C15: 1nF, Capacitor_SMD:C_0805_2012Metric, F.Cu at (154.9, 141.3)
- added C17: 0.1uF, Capacitor_SMD:C_0805_2012Metric, F.Cu at (154.3, 138.1)
- added C2: 0.1uF, Capacitor_SMD:C_0805_2012Metric, F.Cu at (141.7, 141.9)
- added C3: 0.1uF, Capacitor_SMD:C_0805_2012Metric, F.Cu at (148.3, 142.3)
- added D5: MMSZ5222BT1G, Diode_SMD:D_SOD-123, F.Cu at (152.3, 110.6)
- added D6: SMF6.0A, Diode_SMD:D_SOD-123F, F.Cu at (113.4, 131.0)
- added D7: BAT46W-7-F, Diode_SMD:D_SOD-123, F.Cu at (118.4, 121.2)
- added F1: 500mA, Fuse:Fuse_0805_2012Metric, F.Cu at (118.0, 131.0)
- added J1: B1HSW6, Connector_USB:USB_B_OST_USB-B1HSxx_Horizontal, F.Cu at (126.2, 136.4)
- added Q25: 2N7002, Package_TO_SOT_SMD:SOT-23, F.Cu at (155.4, 111.0)
- added R53: 10k+/-0.1%, Resistor_SMD:R_0805_2012Metric, F.Cu at (161.9, 136.4)
- added R54: 1k, Resistor_SMD:R_0805_2012Metric, F.Cu at (141.6, 137.0)
- added R55: 1k, Resistor_SMD:R_0805_2012Metric, F.Cu at (145.5, 137.5)
- added R56: 500, Resistor_SMD:R_0805_2012Metric, F.Cu at (131.4, 126.6)
- added R57: 1k, Resistor_SMD:R_0805_2012Metric, F.Cu at (146.5, 124.1)
- added R58: 1k, Resistor_SMD:R_0805_2012Metric, F.Cu at (145.4, 116.2)
- added R59: 10k, Resistor_SMD:R_0805_2012Metric, F.Cu at (122.1, 123.2)
- added R60: 100k+/-0.1%, Resistor_SMD:R_0805_2012Metric, F.Cu at (138.0, 138.9)
- added R61: 49k+/-0.1%, Resistor_SMD:R_0805_2012Metric, F.Cu at (135.2, 138.2)
- added R62: 10k, Resistor_SMD:R_0805_2012Metric, F.Cu at (149.1, 106.4)
- added R63: 10k, Resistor_SMD:R_0805_2012Metric, F.Cu at (166.0, 100.8)
- added R64: 1k+/-0.1%, Resistor_SMD:R_0805_2012Metric, F.Cu at (135.2, 141.7)
- added R65: 1k+/-0.1%, Resistor_SMD:R_0805_2012Metric, F.Cu at (149.7, 135.7)
- added R66: 50k, Resistor_SMD:R_0805_2012Metric, F.Cu at (131.4, 122.4)
- added R68: 100k, Resistor_SMD:R_0805_2012Metric, F.Cu at (159.0, 108.8)
- added R69: 10k, Resistor_SMD:R_0805_2012Metric, F.Cu at (159.0, 106.7)
- added R7: 10k+/-0.1%, Resistor_SMD:R_0805_2012Metric, F.Cu at (157.5, 129.3)
- added R8: 1.62k, Resistor_SMD:R_0805_2012Metric, F.Cu at (136.7, 130.9)
- added TP5: Pad, TestPoint:TestPoint_THTPad_1.5x1.5mm_Drill0.7mm, F.Cu at (136.7, 126.6)
- added U2: LM4030-2.5, Package_TO_SOT_SMD:SOT-23-5, F.Cu at (133.0, 132.0)
- added U5: TS3A4751PWR, Package_SO:TSSOP-14_4.4x5mm_P0.65mm, F.Cu at (138.0, 121.6)
- added U8: LMV761MF, Package_TO_SOT_SMD:SOT-23-6, F.Cu at (138.4, 141.9)
- added U9: INA326, Package_SO:MSOP-8_3x3mm_P0.65mm, F.Cu at (149.8, 139.4)
- D2: value LTST-C170KRKT -> B340; footprint LED_SMD:LED_0805_2012Metric -> Diode_SMD:D_SMB
- H1, H2, H3, H4: footprint MountingHole:MountingHole_2.7mm_Pad_Via -> MountingHole:MountingHole_3.2mm_M3_Pad_Via
- Q14: value 2N7002 -> BSS84
- R1: value 10k -> 1k+/-0.1%; footprint Resistor_SMD:R_0805_2012Metric_Pad1.20x1.40mm_HandSolder -> Resistor_SMD:R_0805_2012Metric
- R10, R11, R12, R13, R14, R15, R16, R17, R18, R19, R20, R23, R24, R25, R26, R27, R28, R30, R31, R32, R34, R35, R37, R39, R4, R40, R41, R42, R43, R44, R45, R46, R47, R48, R49, R50, R51, R52, R6, R9: footprint Resistor_SMD:R_0805_2012Metric_Pad1.20x1.40mm_HandSolder -> Resistor_SMD:R_0805_2012Metric
- R2: value 10k -> 100k+/-0.1%; footprint Resistor_SMD:R_0805_2012Metric_Pad1.20x1.40mm_HandSolder -> Resistor_SMD:R_0805_2012Metric
- R21: value 100k+/-0.1% -> 10k+/-0.1%; footprint Resistor_SMD:R_0805_2012Metric_Pad1.20x1.40mm_HandSolder -> Resistor_SMD:R_0805_2012Metric
- R22: value 10k -> 500k; footprint Resistor_SMD:R_0805_2012Metric_Pad1.20x1.40mm_HandSolder -> Resistor_SMD:R_0805_2012Metric
- R29: value 649 -> 0; footprint Resistor_SMD:R_0805_2012Metric_Pad1.20x1.40mm_HandSolder -> Resistor_SMD:R_0805_2012Metric
- R3: footprint Capacitor_SMD:C_0805_2012Metric_Pad1.18x1.45mm_HandSolder -> Resistor_SMD:R_0805_2012Metric
- R33: value 1k -> 5k; footprint Resistor_SMD:R_0805_2012Metric_Pad1.20x1.40mm_HandSolder -> Resistor_SMD:R_0805_2012Metric
- R36: value 1.62k -> 10k+/-0.1%; footprint Resistor_SMD:R_0805_2012Metric_Pad1.20x1.40mm_HandSolder -> Resistor_SMD:R_0805_2012Metric
- R38: value 649 -> 10k+/-0.1%; footprint Resistor_SMD:R_0805_2012Metric_Pad1.20x1.40mm_HandSolder -> Resistor_SMD:R_0805_2012Metric
- R5: value 649 -> 10k; footprint Resistor_SMD:R_0805_2012Metric_Pad1.20x1.40mm_HandSolder -> Resistor_SMD:R_0805_2012Metric
- SW1: value GF-123-0054 -> SW_Push; footprint Multimeter:SW_GF-123-0054 -> Button_Switch_THT:SW_PUSH_6mm
- TP4: value 4952 -> Pad; footprint Connector_Pin:Pin_D1.2mm_L10.2mm_W2.9mm_FlatFork -> TestPoint:TestPoint_THTPad_1.5x1.5mm_Drill0.7mm
- moved Q14 69.4 mm to (150.3, 129.0), turned to -90 degrees
- moved D2 68.3 mm to (124.0, 131.0), turned to 0 degrees
- moved R29 60.9 mm to (155.4, 106.7), turned to 0 degrees
- moved R2 55.4 mm to (154.9, 143.4), turned to 0 degrees
- moved R33 53.9 mm to (131.4, 124.5), turned to 0 degrees
- moved J3 52.4 mm to (144.0, 131.0)
- moved R36 48.1 mm to (157.5, 132.8), turned to -90 degrees
- moved J4 48.1 mm to (163.0, 131.0)
- moved R1 47.9 mm to (151.9, 135.7), turned to -90 degrees
- moved TP4 47.3 mm to (125.0, 122.4)
- moved TP1 47.2 mm to (170.6, 125.6)
- moved R38 47.2 mm to (158.4, 136.4), turned to 0 degrees
- moved R42 45.8 mm to (172.1, 120.8), turned to 180 degrees
- moved C6 42.7 mm to (168.8, 113.7)
- moved C5 42.7 mm to (160.4, 120.0)
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Connections:
- net Net-(J4-Pin_1) renamed /Analog Front End/Continuity Detector/Vbias
- J3 pad 1: Net-(J3-Pin_1) -> /Analog Front End/Continuity Detector/Vin
- Q14 pad 2: GND -> Net-(Q14-S)
- Q14 pad 3: Net-(D2-K) -> Net-(D7-A)
- R1 pad 1: +3.3V -> Net-(R1-Pad1)
- R1 pad 2: Net-(U3C-+) -> Net-(R1-Pad2)
- R2 pad 1: Net-(U3C-+) -> Net-(U9-R2)
- R21 pad 1: Net-(SW2A-C) -> REF
- R21 pad 2: Net-(R21-Pad2) -> Net-(U3A-+)
- R22 pad 1: Net-(SW2B-A) -> Net-(U3C--)
- R22 pad 2: +3.3V -> Net-(U5-COM1)
- R29 pad 1: +5V -> Net-(R29-Pad1)
- R29 pad 2: Net-(D2-A) -> Net-(Q25-G)
- R3 pad 2: Net-(SW1-B) -> Net-(U1-TP5_GPIO25/LED)
- R33 pad 1: /Display/pico -> Net-(U3C--)
- R33 pad 2: Net-(Q14-G) -> Net-(U5-COM3)
- R34 pad 1: /Display/nano -> /Display/kilo
- R35 pad 1: /Display/micro -> /Display/mega
- R36 pad 1: +3.3V -> Net-(R36-Pad1)
- R36 pad 2: Net-(U3A-+) -> Net-(R36-Pad2)
- R37 pad 1: Net-(J3-Pin_1) -> /Analog Front End/Continuity Detector/Vin
- R38 pad 1: Net-(SW2A-A) -> Net-(R36-Pad2)
- R38 pad 2: Net-(R21-Pad2) -> Net-(R38-Pad2)
- R5 pad 1: Net-(J3-Pin_1) -> /Analog Front End/current_range1
- R5 pad 2: Net-(R5-Pad2) -> GND
- SW1 pad 1: GND -> Net-(U1-TP5_GPIO25/LED)
- SW1 pad 2: Net-(SW1-B) -> GND
- SW3 pad 3: Net-(R21-Pad2) -> /Analog Front End/Current Source/Iout
- SW3 pad 6: Net-(R5-Pad2) -> /Analog Front End/Continuity Detector/Vin
- SW3 pad 7: unconnected-(SW3-Pad7) -> Net-(R29-Pad1)
- TP3 pad 1: Net-(SW2A-B) -> Net-(C14-Pad1)
- TP4 pad 1: GND -> Net-(U3C--)
- U1 pad 1: unconnected-(U1-GP0-Pad1) -> /Analog Front End/continuity_detected
- U1 pad 11: /Analog Front End/RANGE -> /Analog Front End/current_range2
- U1 pad 12: /Display/low_ohm -> /Analog Front End/current_range3
- U1 pad 14: /Display/micro -> /Analog Front End/current_range4
- U1 pad 15: /Display/nano -> /Display/mega
- U1 pad 16: /Display/pico -> /Display/low_ohm
- U1 pad 2: Net-(SW1-B) -> /Analog Front End/current_range1
- U1 pad 22: unconnected-(U1-GP17-Pad22) -> /Display/kilo
- U1 pad 39: unconnected-(U1-VSYS-Pad39) -> Net-(D6-K)
- U1 pad TP5: unconnected-(U1-TP5_GPIO25/LED-PadTP5) -> Net-(U1-TP5_GPIO25/LED)
- U3 pad 1: Net-(SW2A-B) -> Net-(C14-Pad1)
- U3 pad 10: Net-(U3C-+) -> REF
- U3 pad 2: Net-(SW2A-B) -> Net-(U3A--)
Routing:
- net /Display/micro: track 87.5 -> 0.00 mm, vias 2 -> 0
- net /Display/nano: track 87.0 -> 0.00 mm, vias 2 -> 0
- net /Display/pico: track 83.0 -> 0.00 mm, vias 8 -> 0
- net /Display/D: track 82.4 -> 10.5 mm
- net /Analog Front End/continuity_detected: track 0.00 -> 71.6 mm
- net /Display/C: track 82.3 -> 12.1 mm, vias 2 -> 0
- net Net-(SW2A-B): track 64.5 -> 0.00 mm, vias 6 -> 0
- net Net-(D6-K): track 0.00 -> 63.8 mm
- net /Display/F: track 69.1 -> 6.21 mm, vias 2 -> 0
- net /Display/G: track 65.2 -> 5.61 mm, vias 2 -> 0
- net +5V: track 149.9 -> 90.5 mm, vias 14 -> 16
- net /Analog Front End/Continuity Detector/Vin: track 0.00 -> 56.9 mm
- net /Display/E: track 79.8 -> 24.6 mm
- net Net-(SW1-B): track 50.6 -> 0.00 mm, vias 2 -> 0
- net /Analog Front End/current_range1: track 0.00 -> 47.9 mm
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- removed copper zone on F.Cu, net +5V

Commit message: layout complete
Parts:
- moved R37 0.86 mm to (113.4, 109.7), turned to 90 degrees
- moved R41 0.42 mm to (160.1, 112.7)
- moved R2 0.40 mm to (154.9, 143.0)
- moved C15 0.40 mm to (154.9, 140.9)
- moved C5 0.35 mm to (160.1, 120.0)
- moved R40 0.35 mm to (160.1, 116.3)
Routing:
- net +3.3V: track 26.3 -> 291.9 mm, vias 2 -> 21
- net +5V: track 90.5 -> 137.7 mm, vias 16 -> 9
- net Net-(C14-Pad1): track 8.64 -> 23.6 mm, vias 0 -> 2
- net /Display/C: track 12.1 -> 16.9 mm
- net /Display/D: track 10.5 -> 15.1 mm, vias 2 -> 0
- net /Display/E: track 24.6 -> 28.2 mm
- net Net-(D5-K): track 61.6 -> 58.6 mm
- net GND: track 130.9 -> 133.0 mm
- net /Analog Front End/Continuity Detector/Vbias: track 80.8 -> 81.9 mm
- net /Display/DP: track 25.4 -> 26.4 mm
- net /Analog Front End/MDAT: track 55.5 -> 56.4 mm
- net Net-(U10-CH0): track 23.4 -> 24.1 mm
- net /Analog Front End/SDO: track 61.0 -> 61.7 mm
- net Net-(Q25-D): track 18.6 -> 19.3 mm
- net /Display/A: track 42.2 -> 42.8 mm, vias 2 -> 0
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- removed copper zone on F.Cu, net +3.3V

Commit message: rev3 work
Parts:
- D5: value MMSZ5222BT1G -> DDZ9684-7

Commit message: BOM
Parts:
- C1: value 1uF -> 0.1uF
- R22: value 500k -> 500k+/-0.1%
- R33: value 5k -> 5k+/-0.1%
- R37: value 511k+/-0.1% -> 5.11M+/-1%
- R39: value 10k+/-0.1% -> 100k+/-0.1%
- R56: value 500 -> 499+/-0.1%
- R61: value 49k+/-0.1% -> 50k+/-0.1%
- R66: value 50k -> 50k+/-0.1%
- R68: value 100k -> 100k+/-0.1%
