File: electronics/rev3/ecad/continuity_detector.kicad_sch (KiCad schematic)
At the start: 14 parts, among them U8 LMV761MF, U9 INA326

Commit message: layout work rev3
Parts:
- R1: footprint Capacitor_SMD:C_0805_2012Metric -> Resistor_SMD:R_0805_2012Metric
- R2: footprint (none) -> Resistor_SMD:R_0805_2012Metric
- U8: footprint LMV761MF:SOT95P284X120-6N -> Package_TO_SOT_SMD:SOT-23-6
Changed lines of the file:
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@@
 			)
 		)
-		(property "Footprint" "Capacitor_SMD:C_0805_2012Metric"
+		(property "Footprint" "Resistor_SMD:R_0805_2012Metric"
 			(at 95.504 94.234 90)
 			(effects
@@
 			)
 		)
-		(property "Footprint" "LMV761MF:SOT95P284X120-6N"
+		(property "Footprint" "Package_TO_SOT_SMD:SOT-23-6"
 			(at 177.8 85.09 0)
 			(effects
@@
 			)
 		)
-		(property "Footprint" ""
+		(property "Footprint" "Resistor_SMD:R_0805_2012Metric"
 			(at 129.286 117.094 90)
 			(effects

Commit message: layout complete
Parts:
- C17, C2, C3: Digikey Part # (none) -> 1276-1003-1-ND; Part # (none) -> CL21B104KBCNNNC; Unit Price (none) -> 0.1
Changed lines of the file:
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@@
+			)
+		)
+		(property "Digikey Part #" "1276-1003-1-ND"
+			(at 113.03 76.2 0)
+			(effects
+				(font
+					(size 1.27 1.27)
+				)
+				(hide yes)
+			)
+		)
+		(property "Part #" "CL21B104KBCNNNC"
+			(at 113.03 76.2 0)
+			(effects
+				(font
+					(size 1.27 1.27)
+				)
+				(hide yes)
+			)
+		)
+		(property "Unit Price" "0.1"
+			(at 113.03 76.2 0)
+			(effects
+				(font
+					(size 1.27 1.27)
+				)
+				(hide yes)
 			)
 		)
@@
 		)
 		(property "Description" "Unpolarized capacitor"
+			(at 143.51 81.28 0)
+			(effects
+				(font
+					(size 1.27 1.27)
+				)
+				(hide yes)
+			)
+		)
+		(property "Digikey Part #" "1276-1003-1-ND"
+			(at 143.51 81.28 0)
+			(effects
+				(font
+					(size 1.27 1.27)
+				)
+				(hide yes)
+			)
+		)
+		(property "Part #" "CL21B104KBCNNNC"
+			(at 143.51 81.28 0)
+			(effects
+				(font
+					(size 1.27 1.27)
+				)
+				(hide yes)
+			)
+		)
+		(property "Unit Price" "0.1"
 			(at 143.51 81.28 0)
 			(effects
@@
 			(at 60.96 92.71 0)
 			(effects
+				(font
+					(size 1.27 1.27)
+				)
+				(hide yes)
+			)
+		)
+		(property "Digikey Part #" "1276-1003-1-ND"
+			(at 60.96 92.71 0)
+			(effects
+				(font
+					(size 1.27 1.27)
+				)
+				(hide yes)
+			)
+		)
+		(property "Part #" "CL21B104KBCNNNC"
+			(at 60.96 92.71 0)
+			(effects
+				(font
+					(size 1.27 1.27)
+				)
+				(hide yes)
+			)
+		)
+		(property "Unit Price" "0.1"
+			(at 60.96 92.71 0)
+			(effects

Commit message: rev3 work
Parts:
- R54, R55: Digikey Part # (none) -> RMCF0805FT1K00CT-ND; Part # (none) -> RMCF0805FT1K00; Unit Price (none) -> 0.1
Changed lines of the file:
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@@
+			)
+		)
+		(property "Digikey Part #" "RMCF0805FT1K00CT-ND"
+			(at 55.88 87.63 0)
+			(effects
+				(font
+					(size 1.27 1.27)
+				)
+				(hide yes)
+			)
+		)
+		(property "Part #" "RMCF0805FT1K00"
+			(at 55.88 87.63 0)
+			(effects
+				(font
+					(size 1.27 1.27)
+				)
+				(hide yes)
+			)
+		)
+		(property "Unit Price" "0.1"
+			(at 55.88 87.63 0)
+			(effects
+				(font
+					(size 1.27 1.27)
+				)
+				(hide yes)
 			)
 		)
@@
 			(at 55.88 97.79 0)
 			(effects
+				(font
+					(size 1.27 1.27)
+				)
+				(hide yes)
+			)
+		)
+		(property "Digikey Part #" "RMCF0805FT1K00CT-ND"
+			(at 55.88 97.79 0)
+			(effects
+				(font
+					(size 1.27 1.27)
+				)
+				(hide yes)
+			)
+		)
+		(property "Part #" "RMCF0805FT1K00"
+			(at 55.88 97.79 0)
+			(effects
+				(font
+					(size 1.27 1.27)
+				)
+				(hide yes)
+			)
+		)
+		(property "Unit Price" "0.1"
+			(at 55.88 97.79 0)
+			(effects

Commit message: BOM
Parts:
- C15: Digikey Part # (none) -> 399-C0805C102J5GACTUCT-ND; Part # (none) -> C0805C102J5GACTU; Unit Price (none) -> 0.09
- R1, R64, R65: Digikey Part # (none) -> 541-1.00KCCT-ND; Part # (none) -> CRCW08051K00FKEA; Unit Price (none) -> 0.1
- R2, R60: Digikey Part # (none) -> P10KDACT-ND; Part # (none) -> ERA-6AEB103V; Unit Price (none) -> 0.13
- R61: value 49k+/-0.1% -> 50k+/-0.1%; Digikey Part # (none) -> 749-MCU08050D5002BP100CT-ND; Part # (none) -> MCU08050D5002BP100; Unit Price (none) -> 0.57
- U8: Digikey Part # (none) -> LMV761MFCT-ND; Part # (none) -> LMV761MF; Unit Price (none) -> 3.02
- U9: Digikey Part # (none) -> INA326EA/2K5CT-ND; Part # (none) -> INA326EA/2K5; Unit Price (none) -> 5.05
