File: electronics/rev4/ecad/analog_front _end.kicad_sch (KiCad schematic)
At the start: 22 parts, among them J3 Red Banana Plug, J4 Black Banana Plug, Q25 2N7002, SW3 GF-161-0005, U10 MCP3561, U3 OPA4388IDR

Commit message: stuff
Parts:
- added R70: 649, symbol Device:R_US
- added R71: 10k, symbol Device:R_US
- added TP6: Pad, TestPoint:TestPoint_THTPad_1.5x1.5mm_Drill0.7mm, symbol Connector:TestPoint_Alt
- added U7: CPC1117N, Package_SO:SOP-4_3.8x4.1mm_P2.54mm, symbol Relay_SolidState:CPC1117N
- C1: value 0.1uF -> 1nF
Connections:
- net Current Source/Iout is gone; now on net Continuity Detector/Vin: SW3.3
- net Continuity Detector/Vbias: now also U7.3
- net Continuity Detector/Vin: no longer J3.1 (Pin_1), R37.1, SW3.6
- net GND: now also U7.2
- net at R37.2, SW3.2, SW3.5: now also R71.1, TP6.1, U7.4; no longer D5.1 (K), U3.12 (+)
- new net: J3.1 (Pin_1), R37.1, SW3.6
- new net: D5.1 (K), R71.2, U3.12 (+)
- new net: R70.2, U7.1
- new net zero: R70.1
Other:
- note added: "0.5W"
- moved on the sheet: C1, C4, C5, C6, D5, J3, J4, Q25, R29, R37, R39, R4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

Commit message: work
Parts:
- removed R70: 649, symbol Device:R_US
- removed U7: CPC1117N, Package_SO:SOP-4_3.8x4.1mm_P2.54mm, symbol Relay_SolidState:CPC1117N

Commit message: started rev4
Connections:
- net at C1.1, R39.1, SW3.1: now also R29.1, SW3.7
Other:
- moved on the sheet: Q25, R29, R40, R41, R68, R69
