File: electronics/rev4/ecad/continuity_detector.kicad_sch (KiCad schematic)
At the start: 14 parts, among them U8 LMV761MF, U9 INA326

Commit message: stuff
Parts:
- added C8: 1nF, Capacitor_SMD:C_0805_2012Metric, symbol Device:C
- added R72: R_US, symbol Device:R_US
Connections:
- net GND: now also C8.2
- net at U9.6: now also R72.1; no longer U8.3 (IN-)
- new net: C8.1, R72.2, U8.3 (IN-)
Other:
- moved on the sheet: C15, C17, C3, R1, R2, R54, R55, R65, U9

Commit message: started rev4
Parts:
- removed C3: 0.1uF, Capacitor_SMD:C_0805_2012Metric, symbol Device:C
- removed R55: 1k, Resistor_SMD:R_0805_2012Metric, symbol Device:R_US
- added D8: DDZ9684-7, Diode_SMD:D_SOD-123, symbol Device:D_Zener
Connections:
- net GND: now also D8.2 (A)
- net Vbias: now also U9.2 (-)
- net at R54.2, U9.3 (+): now also D8.1 (K)
Other:
- moved on the sheet: C15, C17, C2, C8, R1, R2, R54, R60, R61, R64, R65, R72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
